File: pcb_capteur_graphite_V2/pcb_capteur_graphite_V2.kicad_pcb (KiCad board)
At the start: 2 copper layers, 68.6 x 53.3 mm, 21 parts, among them J1 Power, J2 Digital/PWM, J3 Analog, J4 Digital/PWM, U1 Blutooth_HC06, U2 LTC1050, U3 capteur, U4 oled

Commit message: version de circuit imprimé
Parts:
- C1, C2, C4: footprint Capacitor_THT:C_Disc_D3.0mm_W1.6mm_P2.50mm -> New_footprints:Conductance
- R1, R2, R3, R4, R5: footprint Resistor_THT:R_Axial_DIN0204_L3.6mm_D1.6mm_P1.90mm_Vertical -> New_footprints:Resistor
- moved U1 7.27 mm to (143.7, 56.8)
- moved U4 5.10 mm to (161.0, 82.7), turned to 0 degrees
- moved C2 2.54 mm to (136.1, 91.9)
- moved R3 2.54 mm to (145.8, 72.1)
- moved C1 2.17 mm to (114.8, 79.4)
- moved R5 1.77 mm to (152.4, 94.0)
- moved R4 1.67 mm to (141.2, 69.1)
- moved R1 1.49 mm to (113.8, 72.6)
Routing:
- net GND: track 71.5 -> 15.1 mm, vias 0 -> 2
- net /SDA/A5: track 29.9 -> 18.3 mm
- net /SCL/A4: track 25.9 -> 17.9 mm
- net /*11/RX: track 16.4 -> 8.75 mm
- net /*10/TX: track 16.4 -> 8.75 mm
- net VCC: track 45.4 -> 50.7 mm
- net Net-(C3-Pad2): track 129.4 -> 130.5 mm, vias 1 -> 2
- net Net-(C3-Pad1): track 22.9 -> 22.1 mm
