File: pcb_capteur_graphite_V2/pcb_capteur_graphite_V2.kicad_sch (KiCad schematic)
At the start: 17 parts, among them J1 Power, J2 Digital/PWM, J3 Analog, J4 Digital/PWM, U1 Blutooth_HC06, U2 LTC1050, U3 capteur, U4 oled

Commit message: version de circuit imprimé
Parts:
- C1, C2, C4: footprint Capacitor_THT:C_Disc_D3.0mm_W1.6mm_P2.50mm -> New_footprints:Conductance
- R1, R2, R3, R4, R5: footprint Resistor_THT:R_Axial_DIN0204_L3.6mm_D1.6mm_P1.90mm_Vertical -> New_footprints:Resistor
Changed lines of the file:
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@@
     (property "Reference" "R5" (id 0) (at 265.43 43.18 90))
     (property "Value" "R" (id 1) (at 265.43 45.72 90))
-    (property "Footprint" "Resistor_THT:R_Axial_DIN0204_L3.6mm_D1.6mm_P1.90mm_Vertical" (id 2) (at 265.43 47.752 90)
+    (property "Footprint" "New_footprints:Resistor" (id 2) (at 265.43 47.752 90)
       (effects (font (size 1.27 1.27)) hide)
     )
@@
       (effects (font (size 1.27 1.27)) (justify left))
     )
-    (property "Footprint" "Capacitor_THT:C_Disc_D3.0mm_W1.6mm_P2.50mm" (id 2) (at 209.2452 59.69 0)
+    (property "Footprint" "New_footprints:Conductance" (id 2) (at 209.2452 59.69 0)
       (effects (font (size 1.27 1.27)) hide)
     )
@@
     (property "Reference" "R1" (id 0) (at 198.12 41.91 90))
     (property "Value" "R" (id 1) (at 198.12 44.45 90))
-    (property "Footprint" "Resistor_THT:R_Axial_DIN0204_L3.6mm_D1.6mm_P1.90mm_Vertical" (id 2) (at 198.12 50.038 90)
+    (property "Footprint" "New_footprints:Resistor" (id 2) (at 198.12 50.038 90)
       (effects (font (size 1.27 1.27)) hide)
     )
@@
       (effects (font (size 1.27 1.27)) (justify right))
     )
-    (property "Footprint" "Resistor_THT:R_Axial_DIN0204_L3.6mm_D1.6mm_P1.90mm_Vertical" (id 2) (at 227.838 55.88 90)
+    (property "Footprint" "New_footprints:Resistor" (id 2) (at 227.838 55.88 90)
       (effects (font (size 1.27 1.27)) hide)
     )
@@
       (effects (font (size 1.27 1.27)) (justify left))
     )
-    (property "Footprint" "Capacitor_THT:C_Disc_D3.0mm_W1.6mm_P2.50mm" (id 2) (at 249.8852 33.02 0)
+    (property "Footprint" "New_footprints:Conductance" (id 2) (at 249.8852 33.02 0)
       (effects (font (size 1.27 1.27)) hide)
     )
@@
       (effects (font (size 1.27 1.27)) (justify right))
     )
-    (property "Footprint" "Resistor_THT:R_Axial_DIN0204_L3.6mm_D1.6mm_P1.90mm_Vertical" (id 2) (at 218.948 55.88 90)
+    (property "Footprint" "New_footprints:Resistor" (id 2) (at 218.948 55.88 90)
       (effects (font (size 1.27 1.27)) hide)
     )
@@
       (effects (font (size 1.27 1.27)) (justify right))
     )
-    (property "Footprint" "Resistor_THT:R_Axial_DIN0204_L3.6mm_D1.6mm_P1.90mm_Vertical" (id 2) (at 259.588 45.72 90)
+    (property "Footprint" "New_footprints:Resistor" (id 2) (at 259.588 45.72 90)
       (effects (font (size 1.27 1.27)) hide)
     )
@@
       (effects (font (size 1.27 1.27)) (justify left))
     )
-    (property "Footprint" "Capacitor_THT:C_Disc_D3.0mm_W1.6mm_P2.50mm" (id 2) (at 272.7452 57.15 0)
+    (property "Footprint" "New_footprints:Conductance" (id 2) (at 272.7452 57.15 0)
       (effects (font (size 1.27 1.27)) hide)
     )
@@
     )
     (path "/51caf9f4-e9f0-4b4a-a71c-590a0bf5400c"
-      (reference "C1") (unit 1) (value "C") (footprint "Capacitor_THT:C_Disc_D3.0mm_W1.6mm_P2.50mm")
+      (reference "C1") (unit 1) (value "C") (footprint "New_footprints:Conductance")
     )
     (path "/7ac8ecad-5c33-4cfb-b1a5-4bc1dafc8002"
-      (reference "C2") (unit 1) (value "C") (footprint "Capacitor_THT:C_Disc_D3.0mm_W1.6mm_P2.50mm")
+      (reference "C2") (unit 1) (value "C") (footprint "New_footprints:Conductance")
     )
     (path "/1261c54b-782f-4308-99b5-9b6287a39cf3"
@@
     )
     (path "/ceaedd2f-69b3-4ee3-8ed8-c8b812f08c4c"
-      (reference "C4") (unit 1) (value "C") (footprint "Capacitor_THT:C_Disc_D3.0mm_W1.6mm_P2.50mm")
+      (reference "C4") (unit 1) (value "C") (footprint "New_footprints:Conductance")
     )
     (path "/00000000-0000-0000-0000-000056d71773"
@@
     )
     (path "/7529285c-d390-4b15-9344-3014868469f9"
-      (reference "R1") (unit 1) (value "R") (footprint "Resistor_THT:R_Axial_DIN0204_L3.6mm_D1.6mm_P1.90mm_Vertical")
+      (reference "R1") (unit 1) (value "R") (footprint "New_footprints:Resistor")
     )
     (path "/8382d94b-2adf-4430-880e-111f987d2d6d"
-      (reference "R2") (unit 1) (value "R") (footprint "Resistor_THT:R_Axial_DIN0204_L3.6mm_D1.6mm_P1.90mm_Vertical")
+      (reference "R2") (unit 1) (value "R") (footprint "New_footprints:Resistor")
     )
     (path "/7605dbe1-b74b-4afa-96d2-236d24d54003"
-      (reference "R3") (unit 1) (value "R") (footprint "Resistor_THT:R_Axial_DIN0204_L3.6mm_D1.6mm_P1.90mm_Vertical")
+      (reference "R3") (unit 1) (value "R") (footprint "New_footprints:Resistor")
     )
     (path "/946c7f90-3f56-4f75-b347-565191e68a04"
-      (reference "R4") (unit 1) (value "R") (footprint "Resistor_THT:R_Axial_DIN0204_L3.6mm_D1.6mm_P1.90mm_Vertical")
+      (reference "R4") (unit 1) (value "R") (footprint "New_footprints:Resistor")
     )
     (path "/129d36cc-4c5a-4d5b-b575-0d267da60b04"
-      (reference "R5") (unit 1) (value "R") (footprint "Resistor_THT:R_Axial_DIN0204_L3.6mm_D1.6mm_P1.90mm_Vertical")
+      (reference "R5") (unit 1) (value "R") (footprint "New_footprints:Resistor")
     )
     (path "/402817ba-818c-4b1f-a552-6395e445d124"
